File: kicad/projects/mixpower-path-mini-axp2585-board-r1/mixpower-path-mini-axp2585-board-r1.kicad_sch (KiCad schematic)
At the start: 83 parts, among them J1 USB_C_USB2.0_16P, J2 BAT, J3 DATA_CONN, J4 PWR_HEADER, J5 DATA_HEADER, Q1 NTLJS7D2P02P8Z, Q2 NTLJS7D2P02P8Z, Q3 NTLJS7D2P02P8Z, Q4 Si1539CDL, Q5 SI2102A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

Commit message: feat: small adjustments to PCB and schem
Parts:
- added FID1, FID2, FID3: Fiducial, Fiducial:Fiducial_0.5mm_Mask1mm, symbol Mechanical:Fiducial
- added R27, R28: 5.1k, Resistor_SMD:R_0402_1005Metric, symbol Device:R_Small
Connections:
- net GND: now also R27.1, R28.1
- net USBC_CC1: now also R28.2
- net USBC_CC2: now also R27.2
Other:
- moved on the sheet: H1, H2, H3, J2, J3, J4, J5, U3
