File: kicad/projects/mixpower-path-mini-bq25672-lv-board-r1/mixpower-path-mini-bq25672-lv-board-r1.kicad_pcb (KiCad board)
At the start: 4 copper layers, 90.9 x 73.6 mm, 165 parts, among them J1 USB_C_Receptacle_HRO_TYPE-C-3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, J2 BAT_HEADERS, J3 BATT, J4 VEXT, J5 PWR_HEADER, J6 DATA_CONN, J7 DATA_HEADER, J8 HAT, J9 DEBUG, Q1 BSS138PS, Q2 DMN3032LFDBQ, Q3 DMN3032LFDBQ, Q4 DMN3032LFDBQ, Q5 SIA931DJ, Q6 SI2101A, Q7 BSS138PS, SW1 TS-A002, SW2 TS-A002, SW3 TS-A002, U1 TL431DBZ, U10 TPS63802, U11 RT9829GQW, U12 TPS63802, U2 TPD8S300A, U3 BQ25672, U4 MAX17055ETB, U5 TPS22917DBV, U6 STM32G071G8U6N, U7 SN74LV1T125DCK, U8 TXS0102DQE, U9 RT9829GQW

Commit message: feat: small changes in schematics, some PCB routing
Parts:
- removed Q5: SIA931DJ, mixlib-generic-dfn:Diodes-Incorporated_U-DFN2020-6_Type-B
- added Q8: NTLJS17D0P03P8Z, mixlib-vendor-onsemi:vendor-onsemi-483av, F.Cu at (198.7, 75.2)
- added REF**: JST_PHD_B12B-PHDSS_2x06_P2.00mm_Vertical, Connector_JST:JST_PHD_B12B-PHDSS_2x06_P2.00mm_Vertical, F.Cu at (160.8, 52.4)
- JP1, TP1, TP4, TP5: moved to B.Cu
- R4, R6: footprint Resistor_SMD:R_0805_2012Metric -> Resistor_SMD:R_0402_1005Metric
- moved C15 98.1 mm to (128.6, 70.9)
- moved D3 97.9 mm to (126.0, 76.9)
- moved C10 97.9 mm to (130.2, 80.8)
- moved C12 97.9 mm to (137.4, 74.0)
- moved C23 97.9 mm to (134.9, 70.2)
- moved C27 97.9 mm to (129.7, 73.9)
- moved C9 97.9 mm to (129.7, 72.9)
- moved L1 97.9 mm to (133.7, 66.8)
- moved Q3 97.9 mm to (129.4, 77.2)
- moved R11 97.9 mm to (131.9, 78.0)
- moved R12 97.9 mm to (131.9, 77.0)
- moved U3 97.9 mm to (133.7, 73.6)
- moved C8 97.9 mm to (119.7, 76.9)
- moved D2 97.9 mm to (121.1, 76.9)
- moved Q2 97.9 mm to (123.6, 77.2)
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Connections:
- net /output-headers/PHER_SCK renamed /output-headers/PHER_GP3_SCK
- net /output-headers/SCL_TX renamed /output-headers/GP2_SCL_TX
- net /output-headers/SDA_RX renamed /output-headers/GP1_SDA_RX
- net /soc-control/~{PHER_EN_GP3} renamed /soc-control/~{PHER_CS}
- D8 pad 4: /soc-control/~{RGB_EN} -> /soc-control/~{RGB_CS}
- J1 pad A6: /input-usb/USBC_D- -> /input-usb/USBC_D+
- J1 pad A7: /input-usb/USBC_D+ -> /input-usb/USBC_D-
- J1 pad B6: /input-usb/USBC_D- -> /input-usb/USBC_D+
- J1 pad B7: /input-usb/USBC_D+ -> /input-usb/USBC_D-
- J8 pad 12: /output-headers/PHER_GP2 -> /output-headers/PHER_GP4
- J8 pad 5: /output-headers/PHER_GP1 -> GND
- R7 pad 1: /input-usb/USBC_D+ -> /input-usb/USBC_D-
- R8 pad 1: /input-usb/USBC_D- -> /input-usb/USBC_D+
- U2 pad 16: unconnected-(U2-D4-Pad16) -> /input-usb/USBC_D+
- U2 pad 17: unconnected-(U2-D3-Pad17) -> /input-usb/USBC_D-
- U6 pad 15: /output-headers/PHER_GP2 -> /soc-control/~{RGB_CS}
- U6 pad 16: /output-headers/PHER_GP1 -> /output-headers/PHER_GP4
Routing:
- net GND: track 25.7 -> 205.8 mm, vias 23 -> 111
- net /input-usb/SHIELD: track 0.00 -> 50.7 mm, vias 0 -> 8
- net /input-usb/VBUS_USBC_IN: track 0.00 -> 47.9 mm, vias 0 -> 12
- net /power-path/VSEL: track 1.88 -> 43.5 mm
- net /power-path/VSYS: track 3.92 -> 44.9 mm
- net /power-path/VBAT: track 12.9 -> 51.4 mm
- net /input-usb/USBC_D-: track 0.00 -> 23.7 mm, vias 0 -> 4
- net /input-usb/USBC_D+: track 0.00 -> 22.5 mm, vias 0 -> 4
- net /power-path/VOTG: track 4.29 -> 25.1 mm
- net /input-usb/USBC_CC2: track 0.00 -> 17.2 mm, vias 0 -> 2
- net /input-usb/USBC_SBU1: track 0.00 -> 16.3 mm, vias 0 -> 2
- net /input-usb/USBC_CC1: track 0.00 -> 15.7 mm
- net /input-vext/VEXT: track 14.3 -> 0.00 mm
- net /soc-control/USBC_CC2: track 0.00 -> 12.5 mm
- net /input-usb/VBUS: track 2.21 -> 14.0 mm
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- added copper zone on F.Cu, net /output-headers/5V
- added copper zone on F.Cu, net /power-path/VSYS
- added copper zone on F.Cu, net /soc-vreg/VSWN_5V_L1
- added copper zone on F.Cu, net /soc-vreg/VSWN_5V_L2
- added copper zone on In1.Cu, net GND
- added copper zone on In2.Cu, net GND

Commit message: feat: failed PCB routing
Parts:
- removed the C14 at (169.2, 28.3)
- removed the C21 at (128.8, 66.5)
- removed the C25 at (138.5, 66.4)
- removed the C27 at (129.7, 73.9)
- removed the C30 at (141.7, 73.4)
- removed the C32 at (182.7, 88.4)
- removed the C33 at (180.1, 90.2)
- removed the C7 at (169.2, 22.4)
- removed the D6 at (192.2, 75.6)
- removed the D8 at (118.0, 32.3)
- removed NT2: 3V3_TO_3V3LP, NetTie:NetTie-2_SMD_Pad0.5mm
- removed the R27 at (175.0, 86.5)
- removed the R28 at (177.6, 87.5)
- removed the R3 at (141.5, 32.0)
- removed the R4 at (141.4, 33.0)
- removed the R5 at (143.8, 37.5)
- removed REF**: JST_PHD_B12B-PHDSS_2x06_P2.00mm_Vertical, Connector_JST:JST_PHD_B12B-PHDSS_2x06_P2.00mm_Vertical
- removed the TP2 at (176.9, 34.8)
- removed the U1 at (140.8, 38.3)
- removed U11: RT9829GQW, mixlib-pmic-supervisor:Specific_DFN8_RT9829_RIT
- removed U12: TPS63802, mixlib-vendor-ti:vendor-ti-DLA0010A
- removed the U4 at (180.8, 87.4)
- added C10: 100n, Capacitor_SMD:C_0402_1005Metric, F.Cu at (130.0, 86.7)
- added C12: 2.2u, Resistor_SMD:R_0402_1005Metric, F.Cu at (200.6, 86.7)
- added C19: 10u, Capacitor_SMD:C_0402_1005Metric, F.Cu at (136.0, 70.1)
- added C23: 10u, Capacitor_SMD:C_0402_1005Metric, F.Cu at (136.0, 71.1)
- added C24: 10u, Capacitor_SMD:C_0402_1005Metric, F.Cu at (140.3, 67.1)
- added C5: 10u, Capacitor_SMD:C_0402_1005Metric, F.Cu at (139.6, 30.0)
- added C56: 10p, Capacitor_SMD:C_0402_1005Metric, F.Cu at (207.6, 57.6)
- added C57: 10p, Capacitor_SMD:C_0402_1005Metric, F.Cu at (207.6, 59.6)
- added C58: 10u, Capacitor_SMD:C_0402_1005Metric, F.Cu at (215.2, 85.8)
- added C59: 470p, Capacitor_SMD:C_0402_1005Metric, F.Cu at (215.2, 87.8)
- added C60: 10u, Capacitor_SMD:C_0402_1005Metric, F.Cu at (215.2, 89.8)
- added C61: 100n, Capacitor_SMD:C_0402_1005Metric, F.Cu at (179.7, 93.7)
- added C8: 2.2u, Capacitor_SMD:C_0402_1005Metric, F.Cu at (112.6, 82.3)
- added C9: 100n, Capacitor_SMD:C_0402_1005Metric, F.Cu at (124.1, 83.9)
- added D4: BZX584C18, Diode_SMD:D_SOD-523, F.Cu at (136.2, 67.9)
- added D7: 1N5817WS, Diode_SMD:D_SOD-323, F.Cu at (204.8, 62.2)
- added JP10: BPROT_DIS, Jumper:SolderJumper-2_P1.3mm_Open_Pad1.0x1.5mm, B.Cu at (116.5, 86.9)
- added JP4: RTC, Jumper:SolderJumper-3_P1.3mm_Open_Pad1.0x1.5mm, F.Cu at (216.7, 60.1)
- added JP5: VDD1_SEL, Jumper:SolderJumper-3_P1.3mm_Open_Pad1.0x1.5mm, F.Cu at (210.9, 86.6)
- added JP9: SHIPFET_DIS, Jumper:SolderJumper-2_P1.3mm_Open_Pad1.0x1.5mm, B.Cu at (116.8, 82.0)
- added Q2: DMN3032LFDBQ, mixlib-generic-dfn:Diodes-Incorporated_U-DFN2020-6_Type-B, F.Cu at (116.4, 82.3)
- added R10: 220, Resistor_SMD:R_0402_1005Metric, F.Cu at (138.4, 35.1)
- added R12: 2, Resistor_SMD:R_0402_1005Metric, F.Cu at (112.6, 80.4)
- added R53: 100k, Resistor_SMD:R_0402_1005Metric, F.Cu at (145.2, 96.9)
- added R54: 100k, Resistor_SMD:R_0402_1005Metric, F.Cu at (154.5, 95.9)
- added R55: 100k, Resistor_SMD:R_0402_1005Metric, F.Cu at (152.5, 95.9)
- added R56: 100k, Resistor_SMD:R_0402_1005Metric, F.Cu at (142.4, 95.9)
- added R57: 100k, Resistor_SMD:R_0402_1005Metric, F.Cu at (144.3, 95.9)
- added R58: 10k, Resistor_SMD:R_0402_1005Metric, F.Cu at (220.1, 51.7)
- added R59: 10k, Resistor_SMD:R_0402_1005Metric, F.Cu at (220.1, 53.7)
- added R60: 1k, Resistor_SMD:R_0402_1005Metric, F.Cu at (220.1, 55.7)
- added R61: 10M, Resistor_SMD:R_0402_1005Metric, F.Cu at (196.0, 51.7)
- added R62: 4.7k, Resistor_SMD:R_0402_1005Metric, F.Cu at (196.0, 53.7)
- added R63: 4.7k, Resistor_SMD:R_0402_1005Metric, F.Cu at (196.0, 55.7)
- added R64: 10M, Resistor_SMD:R_0402_1005Metric, F.Cu at (196.0, 57.7)
- added R65: 4.7k, Resistor_SMD:R_0402_1005Metric, F.Cu at (196.0, 59.7)
- added R66: 4.7k, Resistor_SMD:R_0402_1005Metric, F.Cu at (198.9, 51.7)
- added R67: 4.7k, Resistor_SMD:R_0402_1005Metric, F.Cu at (198.9, 53.7)
- added R68: 0, Resistor_SMD:R_0402_1005Metric, F.Cu at (198.9, 55.7)
- added R69: 0, Resistor_SMD:R_0402_1005Metric, F.Cu at (198.9, 57.7)
- added R7: 220, Resistor_SMD:R_0402_1005Metric, F.Cu at (141.6, 36.1)
- added R70: 0, Resistor_SMD:R_0402_1005Metric, F.Cu at (198.9, 59.7)
- added R71: 0, Resistor_SMD:R_0402_1005Metric, F.Cu at (201.8, 51.7)
- added R72: 0, Resistor_SMD:R_0402_1005Metric, F.Cu at (201.8, 53.7)
- added R73: 0, Resistor_SMD:R_0402_1005Metric, F.Cu at (201.8, 55.7)
- added R74: 10M, Resistor_SMD:R_0402_1005Metric, F.Cu at (214.7, 81.2)
- added R75: 0, Resistor_SMD:R_0402_1005Metric, F.Cu at (214.7, 83.2)
- added R76: 1k, Resistor_SMD:R_0402_1005Metric, F.Cu at (176.8, 90.5)
- added R77: 1M, Resistor_SMD:R_0402_1005Metric, F.Cu at (176.8, 92.5)
- added R78: 4.7k, Resistor_SMD:R_0402_1005Metric, F.Cu at (176.8, 94.5)
- added R79: 1k, Resistor_SMD:R_0402_1005Metric, F.Cu at (176.8, 96.5)
- added R8: 1M, Resistor_SMD:R_0402_1005Metric, F.Cu at (142.5, 36.1)
- added R9: 1.8k, Resistor_SMD:R_1206_3216Metric, F.Cu at (140.3, 31.6)
- added TP4: CC2, TestPoint:TestPoint_Pad_1.0x1.0mm, B.Cu at (142.1, 36.1)
- added TP8: ~{3V3_PG}, TestPoint:TestPoint_Pad_1.0x1.0mm, B.Cu at (149.7, 97.4)
- added U14: TPS7A2601, mixlib-vendor-ti:vendor-ti-DRV0006A-NoThermalVias, F.Cu at (154.5, 111.0)
- added U15: RT9080-33GJ5, Package_TO_SOT_SMD:TSOT-23-5, F.Cu at (158.3, 111.1)
- added U2: FS312F-G, Package_TO_SOT_SMD:SOT-23-6, F.Cu at (121.5, 85.1)
- added U3: MAX17055ETB, mixlib-pmic-battery:SPECIFIC_MAX17055ETB_21-100013A_T102A2&plus_1C_MXM, F.Cu at (128.2, 85.8)
- added Y1: X201232768KJD2SI, Crystal:Crystal_SMD_2012-2Pin_2.0x1.2mm, F.Cu at (200.6, 62.3)
- added Y2: X201624MKB4SI, Crystal:Crystal_SMD_2016-4Pin_2.0x1.6mm, F.Cu at (196.5, 62.5)
- C11: value 100n -> 2.2u
- C13: value 1n -> 10u
- C16, C20, C36, C51: footprint Capacitor_SMD:C_0603_1608Metric -> Capacitor_SMD:C_0402_1005Metric
- C17, C18, C45: value 10u -> 100n; footprint Capacitor_SMD:C_0603_1608Metric -> Capacitor_SMD:C_0402_1005Metric
- C2: renamed from C1; value 2.2u -> 10n
- C25: renamed from C24; value 22u -> 47u
- C26: value 47n -> 47u; footprint Capacitor_SMD:C_0402_1005Metric -> Capacitor_SMD:C_0603_1608Metric
- C29, C47, C52, C53: value 22u -> 10u; footprint Capacitor_SMD:C_0603_1608Metric -> Capacitor_SMD:C_0402_1005Metric
- C30: renamed from C22; footprint Capacitor_SMD:C_0603_1608Metric -> Capacitor_SMD:C_0402_1005Metric
- C31: value 2.2u -> 47n; footprint Capacitor_SMD:C_0603_1608Metric -> Capacitor_SMD:C_0402_1005Metric
- C34: value 2.2u -> 1n; footprint Capacitor_SMD:C_0603_1608Metric -> Capacitor_SMD:C_0402_1005Metric
- C35: value 470p -> 47n
- C37: value 1u -> 10u
- C38: value 10u -> 1n; footprint Capacitor_SMD:C_0603_1608Metric -> Capacitor_SMD:C_0402_1005Metric
- C39: value 10u -> 47u
- C4: renamed from C2; value 2.2u -> 100n
- C40: value 100n -> 47u; footprint Capacitor_SMD:C_0402_1005Metric -> Capacitor_SMD:C_0603_1608Metric
- C46: value 22u -> 100n; footprint Capacitor_SMD:C_0603_1608Metric -> Capacitor_SMD:C_0402_1005Metric
- C50: value 10u -> 100n
- C54: value 100n -> 7p
- C55: value 10u -> 7p
- D1: value TSM24A -> PESD24VV1BA; footprint Package_TO_SOT_SMD:SOT-23 -> Diode_SMD:D_SOD-323
- D2: value BZX384-A10 -> PESD24VV1BA
- D3, D5: value BZX384-A10 -> BZX584C18; footprint Diode_SMD:D_SOD-323 -> Diode_SMD:D_SOD-523
- J3: value BATT -> BATT_JST
- J4: value VEXT -> BATT_PB; footprint Connector_PinHeader_2.54mm:PinHeader_1x02_P2.54mm_Vertical -> Connector_Molex:Molex_PicoBlade_53048-0310_1x03_P1.25mm_Horizontal
- J5: value PWR_HEADER -> VEXT; footprint Connector_PinHeader_2.54mm:PinHeader_1x08_P2.54mm_Vertical -> Connector_PinHeader_2.54mm:PinHeader_1x02_P2.54mm_Vertical
- J6: footprint Connector_JST:JST_ZH_B9B-ZR_1x09_P1.50mm_Vertical -> Connector_Molex:Molex_PicoBlade_53047-1110_1x11_P1.25mm_Vertical
- J7: footprint Connector_PinHeader_2.54mm:PinHeader_1x11_P2.54mm_Vertical -> Connector_PinHeader_2.54mm:PinHeader_1x17_P2.54mm_Vertical
- J8: footprint Connector_IDC:IDC-Header_2x08_P2.54mm_Vertical -> Connector_JST:JST_PHD_B16B-PHDSS_2x08_P2.00mm_Vertical
- JP2: value VDD1_SEL -> RTC; moved to B.Cu
- JP3: footprint Jumper:SolderJumper-3_P1.3mm_Open_RoundedPad1.0x1.5mm -> Jumper:SolderJumper-3_P1.3mm_Open_Pad1.0x1.5mm; moved to B.Cu
- L1: footprint Inductor_SMD:L_Coilcraft_XAL4040-XXX -> Inductor_SMD:L_Coilcraft_XAL4020-XXX
- NT1: value MOSI_TO_RGB_DO -> 3V3_TO_3V3LP; footprint NetTie:NetTie-2_SMD_Pad0.5mm -> NetTie:NetTie-2_SMD_Pad2.0mm
- Q1: value BSS138PS -> DMG1029SVQ; footprint mixlib-generic-sot:SOT-363_SC-70-6 -> mixlib-generic-sot:SOT-563
- Q4: value DMN3032LFDBQ -> NTLJS17D0P03P8Z; footprint mixlib-generic-dfn:Diodes-Incorporated_U-DFN2020-6_Type-B -> mixlib-vendor-onsemi:vendor-onsemi-483av
- Q6: value SI2101A -> DMN3032LFDBQ; footprint mixlib-generic-sot:SOT-323_SC-70 -> mixlib-generic-dfn:Diodes-Incorporated_U-DFN2020-6_Type-B
- Q7: value BSS138PS -> Si1026X; footprint mixlib-generic-sot:SOT-363_SC-70-6 -> mixlib-generic-sot:SOT-563
- Q8: value NTLJS17D0P03P8Z -> DMG1029SVQ; footprint mixlib-vendor-onsemi:vendor-onsemi-483av -> mixlib-generic-sot:SOT-563
- R13: value 100 -> 100k
- R14: value 0 -> 100
- R15: value 0 -> 1k
- R16: value 3k -> 0
- R17: value 2.2k -> 220
- R18: value 1M -> 10k
- R19: value 5.1k -> 0
- R20: value 127k -> 1M
- R21: value 30k -> 0.01; footprint Resistor_SMD:R_0402_1005Metric -> Resistor_SMD:R_1206_3216Metric
- R22: value 100k -> 2
- R23, R34, R50: value 0 -> 100k
- R24: value 2 -> 0; footprint Resistor_SMD:R_0402_1005Metric -> Resistor_SMD:R_0603_1608Metric
- R25: footprint Resistor_SMD:R_0402_1005Metric -> Resistor_SMD:R_0603_1608Metric
- R26, R42: value 1M -> 0
- R29: value 2 -> 2.2k
- R3: renamed from R7; value 22 -> 27
- R30: value 100k -> 1M
- R31: value 1M -> 5.1k
- R32: value 0 -> 30k
- R33: value 1M -> 127k
- R35: value 1M -> 3k
- R36: value 220 -> 100
- R37, R38, R41: value 4.7k -> 0
- R39, R40: value 4.7k -> 10M
- R4: renamed from R8; value 22 -> 27
- R43: value 1M -> 806k
- R44: value 10k -> 91k
- R46: value 806k -> 511k
- R48, R49: value 10k -> 0.01; footprint Resistor_SMD:R_0402_1005Metric -> Resistor_SMD:R_1206_3216Metric
- R51: value 511k -> 100k
- R52: value 91k -> 100k
- TP3: value SOC_RST_PP -> CC1; moved to B.Cu
- TP6: value CC1 -> SOC_RST_PP
- TP7: value CC2 -> ~{5V_PG}; moved to B.Cu
- U10: value TPS63802 -> TPS22917DBV; footprint mixlib-vendor-ti:vendor-ti-DLA0010A -> Package_TO_SOT_SMD:SOT-23-6
- U5: value TPS22917DBV -> TPS63802; footprint Package_TO_SOT_SMD:SOT-23-6 -> mixlib-vendor-ti:vendor-ti-DLA0010A
- U6: value STM32G071G8U6N -> TPS63802; footprint mixlib-vendor-st:QFN-28_4x4mm_P0.5mm -> mixlib-vendor-ti:vendor-ti-DLA0010A
- U7: value SN74LV1T125DCK -> RT9829GQW; footprint Package_TO_SOT_SMD:SOT-353_SC-70-5 -> mixlib-pmic-supervisor:Specific_DFN8_RT9829_RIT
- U8: value TXS0102DQE -> RT9829GQW; footprint Package_SON:X2SON-8_1.4x1mm_P0.35mm -> mixlib-pmic-supervisor:Specific_DFN8_RT9829_RIT
- U9: value RT9829GQW -> STM32G0B1CEU6; footprint mixlib-pmic-supervisor:Specific_DFN8_RT9829_RIT -> Package_DFN_QFN:QFN-48-1EP_7x7mm_P0.5mm_EP5.6x5.6mm
- moved J9 137.2 mm to (220.9, 82.5)
- moved J4 100.8 mm to (96.9, 27.0), turned to -90 degrees
- moved C43 92.7 mm to (212.4, 51.7)
- moved Q7 91.2 mm to (204.3, 65.3)
- moved J5 89.8 mm to (196.8, 88.0), turned to 0 degrees
- moved R37 89.3 mm to (158.3, 104.9)
- moved J3 89.3 mm to (113.8, 23.9)
- moved Q8 87.6 mm to (129.0, 22.0)
- moved R20 87.4 mm to (113.6, 81.5), turned to 90 degrees
- moved J2 86.0 mm to (115.7, 24.3)
- moved U6 85.3 mm to (147.9, 101.5), turned to 180 degrees
- moved R17 84.6 mm to (114.5, 81.5), turned to -90 degrees
- moved R39 84.5 mm to (155.5, 104.9), turned to 180 degrees
- moved TP7 82.8 mm to (157.7, 101.5)
- moved R40 82.5 mm to (159.0, 102.5), turned to -90 degrees
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- renumbered C3 to C1, C15 to C14, C19 to C15, C23 to C21, C28 to C22, C8 to C27, C10 to C28, C6 to C3, C9 to C32, C12 to C33, C4 to C6, C5 to C7, D4 to D6, D7 to D8, Q2 to Q5, R9 to R1, R6 to R11, R10 to R2, R11 to R27, R12 to R28, R1 to R5, R2 to R6, SW3 to SW2, SW2 to SW3, TP4 to TP1, TP5 to TP2, TP1 to TP5, U2 to U1, U3 to U4
Connections:
- C1 pad 1: /input-usb/VCC -> /input-usb/USBC_TPS_VCC
- C11 pad 1: GND -> /input-battery/FG_REG
- C11 pad 2: /input-usb/VBUS -> /input-battery/VBAT_GND
- C13 pad 1: /input-battery/SDRV -> /input-vext/VEXT
- C16 pad 1: /power-path/VSEL -> /power-path/VREGNLP
- C17 pad 1: /power-path/VSEL -> /input-vext/VEXT
- C18 pad 1: /power-path/VSEL -> GND
- C18 pad 2: GND -> /input-usb/VBUS
- C26 pad 1: /power-path/~{CE} -> /power-path/VBAT
- C29 pad 1: /power-path/VBAT -> /power-path/VSEL
- C31 pad 1: /input-battery/VBAT_IN_P -> /power-path/~{CE}
- C31 pad 2: /input-battery/VBAT_IN_GND -> GND
- C34 pad 1: /input-vext/VEXT_P -> /input-battery/SDRV
- C35 pad 1: /vpath-vdd1/VDD1_IN -> /power-path/BC_BATP
- C35 pad 2: /vpath-vdd1/VDD1_CT_G -> GND
- C36 pad 1: /vpath-vdd1/VDD1_IN -> /power-path/VSYS
- C37 pad 1: /soc-control/VDD1_EN -> /power-path/VSYS
- C38 pad 1: /output-headers/VDD1 -> /soc-vreg/VSWREG_5V_EN
- C39 pad 1: /input-usb/VCC -> /soc-vreg/5V_PRE
- C40 pad 1: /input-usb/VCC -> /soc-vreg/3V3_PRE
- C41 pad 1: /util-rgb/VIN_RGB_LP -> /soc-control/SNS_5V_P
- C41 pad 2: /util-rgb/EN_G -> /soc-control/SNS_5V_N
- C42 pad 1: /util-rgb/VIN_RGB_LP -> /soc-control/SNS_3V3_N
- C42 pad 2: GND -> /soc-control/SNS_3V3_P
- C43 pad 1: /input-usb/VCC -> /util-buttons/VPULLUP
- C44 pad 1: /output-headers/VCC -> /util-buttons/VPULLUP
- C45 pad 1: /power-path/VSYS -> /output-headers/~{BTN}
- C46 pad 1: /output-headers/5V -> /output-headers/~{RST}
- C47 pad 1: /output-headers/5V -> /soc-control/BOOT
- C48 pad 1: /output-headers/~{BTN} -> /soc-control/VBAT
- C49 pad 1: /output-headers/VCC -> /soc-control/VREF
- C50 pad 1: /output-headers/BOOT -> /soc-control/3V3LP
- C51 pad 1: /power-path/VSYS -> /soc-control/VBAT
- C52 pad 1: /output-headers/3V3 -> /soc-control/VREF
- C53 pad 1: /output-headers/3V3 -> /soc-control/3V3LP
- C54 pad 1: /output-headers/~{RST} -> GND
- C54 pad 2: GND -> Net-(C54-Pad2)
- C55 pad 1: /input-usb/VBUS -> Net-(C55-Pad1)
- D1 pad 2: GND -> /input-usb/VBUS_USBC_IN
- D2 pad 1: /power-path/VIN1_G -> GND
- D2 pad 2: /power-path/VAC1_MID -> /input-vext/VEXT_IN
- D3 pad 1: /power-path/VIN2_G -> /input-vext/VEXT
- D3 pad 2: /power-path/VAC2_MID -> /input-vext/VEXT_G
- D5 pad 1: /input-vext/VEXT -> /power-path/VIN2_G
- D5 pad 2: /input-vext/VEXT_G -> /power-path/VAC2_MID
- D6 pad 2: Net-(D4-A) -> Net-(D6-A)
- D8 pad 4: /util-rgb/DI_TR -> Net-(D8-DI)
- J4 pad 1: /input-vext/VEXT_IN -> /input-battery/VBAT_IN
- J4 pad 2: GND -> /input-battery/VBAT_IN_GND
- J5 pad 1: /output-headers/5V -> /input-vext/VEXT_IN
- J5 pad 2: /output-headers/3V3 -> GND
- J6 pad 1: /output-headers/GP2_SCL_TX -> /output-headers/USER1_SCL_TX
- J6 pad 3: /output-headers/GP1_SDA_RX -> /output-headers/USER1_SDA_RX
- J6 pad 5: /output-headers/VCC -> /output-headers/3V3
- J7 pad 1: /output-headers/GP2_SCL_TX -> /output-headers/USER1_SCL_TX
- J7 pad 3: /output-headers/GP1_SDA_RX -> /output-headers/USER1_SDA_RX
- J7 pad 5: /output-headers/VCC -> /output-headers/3V3
- J8 pad 11: /soc-control/PHER_SCL_MISO_MCK -> /soc-control/PHER2_MOSI_SCL
- J8 pad 12: /output-headers/PHER_GP4 -> /output-headers/GP1_IRQ2
- J8 pad 13: /output-headers/GP2_SCL_TX -> /soc-control/PHER1_SCL
- J8 pad 14: GND -> /output-headers/GP3
- J8 pad 15: /input-battery/SCL -> /output-headers/USER1_SCL_TX
- J8 pad 2: /input-battery/SDA -> /output-headers/USER1_SDA_RX
- J8 pad 4: /output-headers/GP1_SDA_RX -> /soc-control/PHER1_SDA
- J8 pad 5: GND -> /output-headers/GP4
- J8 pad 6: /~{PHER_IRQ} -> /output-headers/PHER2_SCK
- J8 pad 7: /soc-control/~{PHER_CS} -> /output-headers/GP2
- J8 pad 8: /output-headers/PHER_GP3_SCK -> /input-battery/~{IRQ}
- J8 pad 9: /soc-control/PHER_SDA_MOSI_SD -> /output-headers/PHER2_MISO_SDA
- J9 pad 3: /output-headers/SWCLK -> /soc-control/SWCLK
- JP2 pad 1: /output-headers/3V3 -> /power-path/VBAT
- JP2 pad 2: /vpath-vdd1/VDD1_IN -> /soc-control/VBAT
- JP2 pad 3: /output-headers/5V -> /input-battery/BATP
- JP3 pad 2: /output-headers/VCC -> /util-buttons/VPULLUP
- NT1 pad 1: /soc-control/PHER_SDA_MOSI_SD -> /soc-control/3V3LP
- NT1 pad 2: /soc-control/RGB_DO -> /soc-vreg/3V3_PRE
- Q1 pad 1: Net-(Q1A-S) -> GND
- Q1 pad 2: Net-(Q1A-G) -> /input-usb/DISCH_G
- Q1 pad 3: Net-(Q1B-D) -> /input-usb/USBC_TPS_VCC
- Q1 pad 4: GND -> /soc-control/3V3LP
- Q1 pad 5: /input-usb/DISCH -> Net-(Q1B-G2)
- Q1 pad 6: /input-usb/VBUS -> /input-usb/DISCH_DRAIN
- Q3 pad 1: /power-path/VAC1_MID -> /input-battery/VBAT_GND_RPP
- Q3 pad 2: /power-path/VIN1_G -> /input-battery/BPROT_OD
- Q3 pad 3: /power-path/VSEL -> /input-battery/VBAT_GND_MID
- Q3 pad 4: /power-path/VAC2_MID -> /input-battery/VBAT_GND
- Q3 pad 5: /power-path/VIN2_G -> /input-battery/BPROT_OC
- Q3 pad 6: /power-path/VSEL -> /input-battery/VBAT_GND_MID
- Q3 pad 7: /power-path/VSEL -> /input-battery/VBAT_GND_MID
- Q3 pad 8: /power-path/VSEL -> /input-battery/VBAT_GND_MID
- Q4 pad 1: /input-battery/VBAT_GND -> /input-vext/VEXT_IN
- Q4 pad 2: /input-battery/VBAT_IN_RPP_G -> /input-vext/VEXT_IN
- Q4 pad 3: /input-battery/VBAT_IN -> /input-vext/VEXT_G
- Q4 pad 4: /power-path/VBAT -> /input-vext/VEXT
- Q4 pad 5: Net-(Q4B-G2) -> /input-vext/VEXT_IN
- Q4 pad 6: /input-battery/VBAT_IN_GND -> /input-vext/VEXT_IN
- Q4 pad 7: /input-battery/VBAT_IN_GND -> /input-vext/VEXT_IN
- Q4 pad 8: /input-battery/VBAT_IN -> /input-vext/VEXT
- Q5 pad 3: /input-usb/VBUS -> /power-path/VSEL
- Q5 pad 4: /power-path/VAC2_MID -> /power-path/VAC1_MID
- Q5 pad 5: /power-path/VIN2_G -> /power-path/VIN1_G
- Q5 pad 8: /input-usb/VBUS -> /power-path/VSEL
- Q6 pad 1: /util-rgb/EN_G -> /power-path/VAC2_MID
- Q6 pad 2: /output-headers/5V -> /power-path/VIN2_G
- Q6 pad 3: /util-rgb/VIN_RGB_LP -> /power-path/VSEL
- Q8 pad 1: /input-vext/VEXT_IN -> /soc-control/PHER2_RGB_DO
- Q8 pad 2: /input-vext/VEXT_IN -> /soc-control/PHER2_RGB_CS
- Q8 pad 3: /input-vext/VEXT_G -> /util-rgb/VIN_RGB_LP
- Q8 pad 4: /input-vext/VEXT -> /output-headers/5V
- Q8 pad 5: /input-vext/VEXT_IN -> /util-rgb/EN_G
- Q8 pad 6: /input-vext/VEXT_IN -> Net-(D8-DI)
- R13 pad 1: /input-battery/BATP -> /input-battery/VBAT_IN
- R13 pad 2: /power-path/BC_BATP -> /input-battery/VBAT_IN_RPP_G
- R14 pad 1: Net-(U3-~{QON}) -> /input-battery/VBAT_IN
- R14 pad 2: /output-headers/~{BTN} -> /input-battery/BPROT_VCC
- R15 pad 1: Net-(U3-~{QON}) -> /input-battery/BPROT_CS
- R15 pad 2: GND -> /input-battery/VBAT_GND
- R16 pad 1: GND -> /input-battery/BATP
- R16 pad 2: /power-path/BC_PROG -> /input-battery/VBAT_IN
- R17 pad 1: Net-(D4-A) -> /input-battery/SDRV
- R17 pad 2: /power-path/VREGNLP -> /input-battery/SHIPFET_G
- R18 pad 1: /power-path/~{CE} -> /input-battery/FG_THRM
- R18 pad 2: /power-path/VREGNLP -> /input-battery/FG_AIN
- R19 pad 1: /power-path/TS -> /input-battery/FG_AIN
- R19 pad 2: /power-path/VREGNLP -> /power-path/TS
- R20 pad 1: /power-path/BC_ILIM -> /input-battery/SDRV
- R20 pad 2: /power-path/VREGNLP -> GND
- R21 pad 1: GND -> /input-battery/VBAT_GND
- R21 pad 2: /power-path/TS -> GND
- R22 pad 1: GND -> /input-vext/VEXT_IN
- R22 pad 2: /power-path/BC_ILIM -> /input-vext/VEXT_FLT_P
- R23 pad 1: /input-battery/BATP -> /input-vext/VEXT_G
- R23 pad 2: /input-battery/VBAT_IN -> GND
- R24 pad 1: /input-battery/VBAT_IN -> /power-path/BC_D+
- R24 pad 2: /input-battery/VBAT_IN_P -> /output-headers/D+
- R25 pad 1: /input-battery/SDRV -> /power-path/BC_D-
- R25 pad 2: Net-(Q4B-G2) -> /output-headers/D-
- R26 pad 1: Net-(Q4B-G2) -> /power-path/~{BC_QON}
- R26 pad 2: GND -> /output-headers/~{BTN}
- R29 pad 1: /input-vext/VEXT_IN -> Net-(D6-A)
- R29 pad 2: /input-vext/VEXT_P -> /power-path/VREGNLP
- R30 pad 1: /input-vext/VEXT_G -> /power-path/~{CE}
- R30 pad 2: GND -> /power-path/VREGNLP
- R31 pad 1: /vpath-vdd1/VDD1_IN -> /power-path/TS
- R31 pad 2: /soc-control/VDD1_EN -> /power-path/VREGNLP
- R32 pad 1: /vpath-vdd1/VDD1_QOD_G -> GND
- R32 pad 2: /output-headers/VDD1 -> /power-path/TS
- R33 pad 1: /soc-control/VDD1_EN -> /power-path/BC_ILIM
- R33 pad 2: GND -> /power-path/VREGNLP
- R34 pad 1: /output-headers/SWCLK -> GND
- R34 pad 2: /output-headers/BOOT -> /power-path/BC_ILIM
- R35 pad 1: /output-headers/5V -> GND
- R35 pad 2: /util-rgb/EN_G -> /power-path/BC_PROG
- R36 pad 1: /util-rgb/EN_G -> /input-battery/BATP
- R36 pad 2: /soc-control/~{RGB_EN} -> /power-path/BC_BATP
- R37 pad 1: /output-headers/VCC -> /soc-vreg/VSWREG_5V_EN
- R37 pad 2: /output-headers/GP2_SCL_TX -> /soc-control/5V_EN
- R38 pad 1: /output-headers/VCC -> /soc-vreg/VSWREG_3V3_MODE
- R38 pad 2: /output-headers/GP1_SDA_RX -> /soc-control/SWREG_MODE
- R39 pad 1: /output-headers/VCC -> /soc-vreg/VSWREG_5V_EN
- R39 pad 2: /~{PHER_IRQ} -> /power-path/VSYS
- R40 pad 1: /output-headers/VCC -> GND
- R40 pad 2: /output-headers/~{IRQB} -> /soc-control/SWREG_MODE
- R41 pad 1: /input-usb/VCC -> GND
- R41 pad 2: Net-(D8B-A2) -> /soc-vreg/VSWREG_3V3_MODE
- R42 pad 1: /soc-control/FRSTX1 -> Net-(R42-Pad1)
- R42 pad 2: GND -> /soc-vreg/5V_PRE
- R43 pad 1: /soc-control/FRSTX2 -> /soc-vreg/VSWREG_5V_FB
- R43 pad 2: GND -> Net-(R42-Pad1)
- R44 pad 1: /output-headers/VCC -> GND
- R44 pad 2: /output-headers/~{BTN} -> /soc-vreg/VSWREG_5V_FB
- R45 pad 2: /output-headers/5V -> /soc-vreg/3V3_PRE
- R46 pad 1: /soc-vreg/VSWREG_FB -> /soc-vreg/VSWREG_3V3_FB
- R47 pad 2: /soc-vreg/VSWREG_FB -> /soc-vreg/VSWREG_3V3_FB
- R48 pad 1: /output-headers/VCC -> /soc-vreg/5V_PRE
- R48 pad 2: /output-headers/~{RST} -> /output-headers/5V
- R49 pad 1: /output-headers/BOOT -> /soc-vreg/3V3_PRE
- R49 pad 2: GND -> /output-headers/3V3
- R50 pad 1: Net-(R50-Pad1) -> /soc-control/SNS_5V_P
- R50 pad 2: /output-headers/3V3 -> /soc-vreg/5V_PRE
- R51 pad 1: /soc-vreg/VSWREG_FB -> /soc-control/SNS_5V_N
- R51 pad 2: Net-(R50-Pad1) -> /output-headers/5V
- R52 pad 1: GND -> /soc-control/SNS_3V3_N
- R52 pad 2: /soc-vreg/VSWREG_FB -> /output-headers/3V3
- SW3 pad 1: /output-headers/VCC -> /util-buttons/VPULLUP
- SW3 pad 2: /output-headers/BOOT -> /soc-control/BOOT
- TP3 pad 1: /util-buttons/SRST_BOOT_RST1 -> /soc-control/USBC_CC1
- TP6 pad 1: /soc-control/USBC_CC1 -> /util-buttons/SRST_RST_RST2
- TP7 pad 1: /soc-control/USBC_CC2 -> /soc-vreg/VSWREG_5V_PG
- U1 pad 10: /input-usb/VCC -> /input-usb/USBC_TPS_VCC
- U10 pad 1: /power-path/VSYS -> /vpath-vdd1/VDD1_IN
- U10 pad 3: GND -> /soc-control/VDD1_EN
- U10 pad 4: /soc-vreg/VSWREG_FB -> /vpath-vdd1/VDD1_CT_G
- U10 pad 5: unconnected-(U10-PG-Pad5) -> /vpath-vdd1/VDD1_QOD_G
- U10 pad 6: /output-headers/5V -> /output-headers/VDD1
- U4 pad 12: Net-(U3-~{QON}) -> /power-path/~{BC_QON}
- U4 pad 14: /input-battery/SCL -> /soc-control/PHER1_SCL
- U4 pad 15: /input-battery/SDA -> /soc-control/PHER1_SDA
- U4 pad 21: /~{PHER_IRQ} -> /input-battery/~{IRQ}
- U4 pad 6: /output-headers/D+ -> /power-path/BC_D+
- U4 pad 7: /output-headers/D- -> /power-path/BC_D-
- U5 pad 1: /vpath-vdd1/VDD1_IN -> /soc-vreg/VSWREG_5V_EN
- U5 pad 2: GND -> /soc-control/SWREG_MODE
- U5 pad 3: /soc-control/VDD1_EN -> GND
- U5 pad 4: /vpath-vdd1/VDD1_CT_G -> /soc-vreg/VSWREG_5V_FB
- U5 pad 5: /vpath-vdd1/VDD1_QOD_G -> /soc-vreg/VSWREG_5V_PG
- U5 pad 6: /output-headers/VDD1 -> /soc-vreg/5V_PRE
- U6 pad 1: /input-usb/~{FLT} -> /power-path/VSYS
- U6 pad 10: /soc-control/~{PHER_CS} -> /power-path/VSYS
- U6 pad 2: /soc-control/~{RGB_EN} -> /soc-vreg/VSWREG_3V3_MODE
- U6 pad 3: /input-usb/VCC -> GND
- U6 pad 4: GND -> /soc-vreg/VSWREG_3V3_FB
- U6 pad 5: /output-headers/~{RST} -> /soc-vreg/VSWREG_3V3_PG
- U6 pad 6: /soc-control/FRSTX1 -> /soc-vreg/3V3_PRE
- U6 pad 7: /soc-control/VDD1_EN -> /soc-vreg/VSWN_3V3_L2
- U6 pad 8: /power-path/~{CE} -> GND
- U6 pad 9: /soc-control/FRSTX2 -> /soc-vreg/VSWN_3V3_L1
- U7 pad 1: GND -> /util-buttons/SRST_RST_RST2
- U7 pad 2: /soc-control/RGB_DO -> GND
- U7 pad 3: GND -> /output-headers/~{BTN}
- U7 pad 4: /util-rgb/DI_TR -> /output-headers/~{RST}
- U7 pad 5: /util-rgb/VIN_RGB_LP -> GND
- U8 pad 1: /input-usb/VCC -> /util-buttons/SRST_BOOT_RST2
- U8 pad 2: /input-battery/SDA -> GND
- U8 pad 3: /input-battery/SCL -> /output-headers/~{RST}
- U8 pad 4: GND -> /util-buttons/SRST_BOOT_RST1
- U8 pad 5: Net-(D8B-A2) -> GND
- U8 pad 6: /soc-control/PHER_SCL_MISO_MCK -> unconnected-(U8-NC-Pad6)
- U8 pad 7: /soc-control/PHER_SDA_MOSI_SD -> GND
- U8 pad 8: /input-usb/VCC -> /util-buttons/VPULLUP
- U9 pad 1: /util-buttons/SRST_RST_RST2 -> /input-battery/~{IRQ}
- U9 pad 2: GND -> /soc-control/OSC32_IN
- U9 pad 3: /output-headers/~{BTN} -> /soc-control/OSC32_OUT
- U9 pad 4: /output-headers/~{RST} -> /soc-control/VBAT
- U9 pad 5: GND -> /soc-control/VREF
- U9 pad 6: unconnected-(U9-NC-Pad6) -> /soc-control/3V3LP
- U9 pad 8: /output-headers/VCC -> /soc-control/OSC_IN
Routing:
- net GND: track 205.8 -> 267.6 mm, vias 111 -> 123
- net /power-path/VSYS: track 44.9 -> 89.3 mm, vias 0 -> 6
- net /power-path/VAC2_MID: track 0.00 -> 43.3 mm, vias 0 -> 8
- net /input-vext/VEXT: track 0.00 -> 43.1 mm, vias 0 -> 6
- net /power-path/VSEL: track 43.5 -> 83.6 mm
- net /power-path/VBAT: track 51.4 -> 89.3 mm, vias 8 -> 7
- net /input-battery/VBAT_GND: track 6.62 -> 44.4 mm, vias 0 -> 6
- net /power-path/VAC1_MID: track 0.00 -> 28.9 mm, vias 0 -> 8
- net /input-usb/VBUS: track 14.0 -> 42.8 mm, vias 0 -> 5
- net /power-path/VIN1_G: track 0.00 -> 28.2 mm, vias 0 -> 3
- net /output-headers/D-: track 4.61 -> 30.0 mm
- net /power-path/VIN2_G: track 0.00 -> 25.0 mm, vias 0 -> 3
- net /output-headers/D+: track 4.76 -> 29.3 mm
- net /input-battery/VBAT_IN: track 6.69 -> 31.1 mm, vias 0 -> 6
- net /soc-vreg/3V3_PRE: track 0.00 -> 22.4 mm
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- removed copper zone on F.Cu, net /output-headers/5V
- removed copper zone on F.Cu, net /power-path/VSYS
- removed copper zone on F.Cu, net /soc-vreg/VSWN_5V_L1
- removed copper zone on F.Cu, net /soc-vreg/VSWN_5V_L2
- removed copper zone on F.Cu, net GND
