File: kicad/projects/mixpower-path-mini-bq25672-lv-board-r1/mixpower-path-mini-bq25672-lv-board-r1.kicad_sch (KiCad schematic)
At the start: 0 parts

Commit message: feat: failed PCB routing
Connections:
- no-connect marks 3 -> 15
Other:
- added sheet vpath-vdd2 (sheets/vpath-vdd2.kicad_sch)
- added sheet vpath-vdd2-multi (vpath-vdd2.kicad_sch)
- sheet input-battery ports: added RTC_VBAT; removed none
- sheet input-usb ports: added VCC_DIS; removed none
- sheet output-headers ports: added GP1_IRQ2, GP2, GP3, GP4, PHER1_SCL, PHER1_SDA, PHER2_MISO_SDA, PHER2_MOSI_SCL, PHER2_SCK, USER1_SCL_TX, USER1_SDA_RX, VBAT, VSEL, ~{PHER1_IRQ1}; removed GP1_SDA_RX, GP2_SCL_TX, PHER_GP3_SCK, PHER_GP4, PHER_SCL, PHER_SCL_MISO_MCK, PHER_SDA, PHER_SDA_MOSI_SD, VCC, ~{PHER_CS}, ~{PHER_IRQ}
- sheet power-path ports: added none; removed VCC
- sheet soc-control ports: added 5V_EN, GP1_IRQ2, GP2, GP3, GP4, PHER1_SCL, PHER1_SDA, PHER2_MISO_SDA, PHER2_MOSI_SCL, PHER2_RGB_CS, PHER2_RGB_DO, PHER2_SCK, SNS_3V3_N, SNS_3V3_P, SNS_5V_N, SNS_5V_P, SWREG_MODE, USBC_VCC_DIS, USB_D+, USB_D-, USER1_SCL_TX, USER1_SDA_RX, VBAT, VPULLUP, ~{PHER1_IRQ1}, ~{PHER2_RGB_EN}, ~{SNS_EN}; removed GP1_SDA_RX, GP2_SCL_TX, PHER_GP3_SCK, PHER_GP4, PHER_SCL, PHER_SCL_MISO_MCK, PHER_SDA, PHER_SDA_MOSI_SD, RGB_DO, VCC, ~{PHER_CS}, ~{PHER_IRQ}, ~{RGB_EN}
- sheet soc-vreg ports: added 5V_EN, SNS_3V3_N, SNS_3V3_P, SNS_5V_N, SNS_5V_P, SWREG_MODE, VPULLUP, ~{SNS_EN}; removed VCC
- sheet util-buttons ports: added USER_BOOT, VPULLUP; removed VCC
- sheet util-rgb ports: added 3V3_CS; removed none
- sheet vpath-vdd1 ports: added VDD1; removed VOUT
- note added: "Follow left-to-right"
- note added: "PPC & BC"
- note added: "USB-PD / BATTERY / EXTERNAL POWER PATH CHARGER BOARD"
- note removed: "PPC BC"
