File: kicad/projects/mixpower-path-mini-bq25672-lv-board-r1/sheets/power-path.kicad_sch (KiCad schematic)
At the start: 44 parts, among them Q2 DMN3032LFDBQ, Q3 DMN3032LFDBQ, U3 BQ25672

Commit message: feat: small changes in schematics, some PCB routing
Parts:
- removed R53: 0, Resistor_SMD:R_0402_1005Metric, symbol Device:R_Small
Changed lines of the file:
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@@
 	)
 	(junction
-		(at 92.71 99.06)
-		(diameter 0)
-		(color 0 0 0 0)
-	)
-	(junction
 		(at 52.07 72.39)
 		(diameter 0)
@@
 	(wire
 		(pts
-			(xy 92.71 107.95) (xy 102.87 107.95)
-		)
-		(stroke
-			(width 0)
-			(type default)
-		)
-	)
-	(wire
-		(pts
 			(xy 87.63 41.91) (xy 87.63 72.39)
 		)
@@
 	(wire
 		(pts
-			(xy 92.71 105.41) (xy 92.71 107.95)
-		)
-		(stroke
-			(width 0)
-			(type default)
-		)
-	)
-	(wire
-		(pts
 			(xy 52.07 60.96) (xy 52.07 57.15)
 		)
@@
 	(wire
 		(pts
-			(xy 85.09 99.06) (xy 92.71 99.06)
-		)
-		(stroke
-			(width 0)
-			(type default)
-		)
-	)
-	(wire
-		(pts
 			(xy 45.72 129.54) (xy 45.72 132.08)
 		)
@@
 	(wire
 		(pts
-			(xy 92.71 99.06) (xy 92.71 100.33)
-		)
-		(stroke
-			(width 0)
-			(type default)
-		)
-	)
-	(wire
-		(pts
 			(xy 121.92 54.61) (xy 123.19 54.61)
 		)
@@
 	(wire
 		(pts
-			(xy 92.71 99.06) (xy 93.98 99.06)
+			(xy 85.09 99.06) (xy 93.98 99.06)
 		)
 		(stroke
@@
 		)
 	)
-	(label "VCC"
-		(at 102.87 107.95 180)
-		(effects
-			(font
-				(size 1.016 1.016)
-			)
-			(justify right bottom)
-		)
-	)
 	(label "TS"
 		(at 138.43 130.81 180)
@@
 		)
 		(instances
-			(project ""
+			(project "mixpower-path-mini-bq25672-lv-board-r1"
 				(path "/2e43857b-9bf9-460c-948c-ec2cf8a8d6b4/62cc8ba8-a4a6-4ef3-833b-8755302cfb85"
 					(reference "Q2")
@@
 	)
 	(symbol
-		(lib_id "Device:R_Small")
-		(at 92.71 102.87 0)
-		(unit 1)
-		(exclude_from_sim no)
-		(in_bom yes)
-		(on_board yes)
-		(dnp yes)
-		(fields_autoplaced yes)
-		(property "Reference" "R53"
-			(at 95.25 101.5999 0)
-			(effects
-				(font
-					(size 1.016 1.016)
-				)
-				(justify left)
-			)
-		)
-		(property "Value" "0"
-			(at 95.25 104.1399 0)
-			(effects
-				(font
-					(size 1.016 1.016)
-				)
-				(justify left)
-			)
-		)
-		(property "Footprint" "Resistor_SMD:R_0402_1005Metric"
-			(at 92.71 102.87 0)
-			(effects
-				(font
-					(size 1.27 1.27)
-				)
-				(hide yes)
-			)
-		)
-		(property "Datasheet" "~"
-			(at 92.71 102.87 0)
-			(effects
-				(font
-					(size 1.27 1.27)
-				)
-				(hide yes)
-			)
-		)
-		(property "Description" "Resistor, small symbol"
-			(at 92.71 102.87 0)
-			(effects
-				(font
-					(size 1.27 1.27)
-				)
-				(hide yes)
-			)
-		)
-		(pin "2"
-		)
-		(pin "1"
-		)
-		(instances
-			(project "mixpower-path-mini-bq25672-lv-board-r1"
-				(path "/2e43857b-9bf9-460c-948c-ec2cf8a8d6b4/62cc8ba8-a4a6-4ef3-833b-8755302cfb85"
-					(reference "R53")
-					(unit 1)
-				)
-			)
-		)
-	)
-	(symbol
 		(lib_id "power:GND")
 		(at 30.48 57.15 0)
@@
 		)
 		(instances
-			(project ""
+			(project "mixpower-path-mini-bq25672-lv-board-r1"
 				(path "/2e43857b-9bf9-460c-948c-ec2cf8a8d6b4/62cc8ba8-a4a6-4ef3-833b-8755302cfb85"
 					(reference "U3")
@@
 		)
 		(instances
-			(project ""
+			(project "mixpower-path-mini-bq25672-lv-board-r1"
 				(path "/2e43857b-9bf9-460c-948c-ec2cf8a8d6b4/62cc8ba8-a4a6-4ef3-833b-8755302cfb85"
 					(reference "L1")

Commit message: feat: failed PCB routing
Parts:
- removed C17, C18, C21: 10u, Capacitor_SMD:C_0603_1608Metric, symbol Device:C_Small
- removed C25, C30: 22u, Capacitor_SMD:C_0603_1608Metric, symbol Device:C_Small
- removed C27: 10u, Capacitor_SMD:C_0402_1005Metric, symbol Device:C_Small
- removed D2, D3: BZX384-A10, Diode_SMD:D_SOD-323, symbol Diode:BZX384xxxx
- removed unit 2 of Q2
- removed Q3: DMN3032LFDBQ, mixlib-generic-dfn:Diodes-Incorporated_U-DFN2020-6_Type-B, symbol mixlib-discrete-mosfet:DMN3032LFDBQ
- removed R15: 0, Resistor_SMD:R_0402_1005Metric, symbol Device:R_Small
- added C19, C23, C24: 10u, Capacitor_SMD:C_0402_1005Metric, symbol Device:C_Small
- added C26: 47u, Capacitor_SMD:C_0603_1608Metric, symbol Device:C_Small
- added D4, D5: BZX584C18, Diode_SMD:D_SOD-523, symbol Diode:DZ2S180X0L
- added unit 2 of Q5
- added Q6: DMN3032LFDBQ, mixlib-generic-dfn:Diodes-Incorporated_U-DFN2020-6_Type-B, symbol mixlib-discrete-mosfet:DMN3032LFDBQ
- added R24, R25: 0, Resistor_SMD:R_0603_1608Metric, symbol Device:R_Small
- C16, C20: footprint Capacitor_SMD:C_0603_1608Metric -> Capacitor_SMD:C_0402_1005Metric; Voltage (none) -> 35V
- C25: renamed from C24; value 22u -> 47u; Voltage (none) -> 25V
- C29: value 22u -> 10u; footprint Capacitor_SMD:C_0603_1608Metric -> Capacitor_SMD:C_0402_1005Metric; Voltage (none) -> 35V
- C30: renamed from C22; footprint Capacitor_SMD:C_0603_1608Metric -> Capacitor_SMD:C_0402_1005Metric; Voltage (none) -> 35V
- L1: footprint Inductor_SMD:L_Coilcraft_XAL4040-XXX -> Inductor_SMD:L_Coilcraft_XAL4020-XXX
- renumbered C15 to C14, C19 to C15, C7 to C17, C11 to C18, C23 to C21, C28 to C22, C8 to C27, C10 to C28, C26 to C31, C9 to C32, C12 to C33, C13 to C34, C14 to C35, D4 to D6, Q2 to Q5, R14 to R26, R11 to R27, R12 to R28, R17 to R29, R18 to R30, R19 to R31, R21 to R32, R20 to R33, R22 to R34, R16 to R35, R13 to R36, U3 to U4
Connections:
- net D+: now also R24.2; no longer U4.6 (D+)
- net D-: now also R25.2; no longer U4.7 (D-)
- net GND: now also C19.2, C23.2, C24.2, C26.2
- net VAC1_MID: now also D4.2 (A), Q5.4 (S2)
- net VAC2: now also Q6.6 (D1), Q6.7 (D1)
- net VAC2_MID: now also D5.2 (A), Q6.1 (S1), Q6.4 (S2)
- net VBAT: now also C26.1; no longer C29.1
- net VIN1_G: now also D4.1 (K), Q5.5 (G2)
- net VIN2_G: now also D5.1 (K), Q6.2 (G1), Q6.5 (G2)
- net VOTG: now also C24.1
- net VREGNLP: now also C16.1
- net VSEL: now also C29.1, C19.1, C23.1, Q5.3 (D2), Q5.8 (D2), Q6.3 (D2), Q6.8 (D2); no longer C16.1
- net ~{BC_QON}: now reaches R26.1, U4.12 (~{QON})
- new net BC_D+: R24.1, U4.6 (D+)
- new net BC_D-: R25.1, U4.7 (D-)
Other:
- note added: "* Switching nodes. Place them near each other. * Assuming: Iripple = 2.5A Iinput = 3A Icharge = 3A Isat = 3+(2.5/2) = 4.25A"
- note removed: "* Just a safeguard in case my ~{QON} logic ends up not working out. * Remove the series resistor to disable ~{QON} control."
- note removed: "* Switching nodes. Place them near each other."
- moved on the sheet: C14, C15, C21, C22, C25, C30, R29, R30, R31, R33
