File: kicad/projects/mixpower-path-mini-bq25672-lv-board-r1/sheets/soc-vreg.kicad_sch (KiCad schematic)
At the start: 18 parts, among them U10 TPS63802, U12 TPS63802

Commit message: feat: failed PCB routing
Parts:
- removed C46, C47, C52, C53: 22u, Capacitor_SMD:C_0603_1608Metric, symbol Device:C_Small
- added C38: 1n, Capacitor_SMD:C_0402_1005Metric, symbol Device:C_Small
- added C39, C40: 47u, Capacitor_SMD:C_0603_1608Metric, symbol Device:C_Small
- added C41, C42: 100n, Capacitor_SMD:C_0402_1005Metric, symbol Device:C_Small
- added R37, R38, R41: 0, Resistor_SMD:R_0402_1005Metric, symbol Device:R_Small
- added R39, R40: 10M, Resistor_SMD:R_0402_1005Metric, symbol Device:R_Small
- added R48, R49: 0.01, Resistor_SMD:R_1206_3216Metric, symbol Device:R_Small
- added R50, R51, R52, R53, R54, R55, R56, R57: 100k, Resistor_SMD:R_0402_1005Metric, symbol Device:R_Small
- added TP7: ~{5V_PG}, TestPoint:TestPoint_Pad_1.0x1.0mm, symbol Connector:TestPoint_Small
- added TP8: ~{3V3_PG}, TestPoint:TestPoint_Pad_1.0x1.0mm, symbol Connector:TestPoint_Small
- added U14: TPS7A2601, mixlib-vendor-ti:vendor-ti-DRV0006A-NoThermalVias, symbol mixlib-pmic-vreg:TPS7A2601
- added U15: RT9080-33GJ5, Package_TO_SOT_SMD:TSOT-23-5, symbol mixlib-pmic-vreg:RT9080
- C36: renamed from C45; footprint Capacitor_SMD:C_0603_1608Metric -> Capacitor_SMD:C_0402_1005Metric
- C37: renamed from C51; footprint Capacitor_SMD:C_0603_1608Metric -> Capacitor_SMD:C_0402_1005Metric
- JP3: footprint Jumper:SolderJumper-3_P1.3mm_Open_RoundedPad1.0x1.5mm -> Jumper:SolderJumper-3_P1.3mm_Open_Pad1.0x1.5mm
- NT1: renamed from NT2; footprint NetTie:NetTie-2_SMD_Pad0.5mm -> NetTie:NetTie-2_SMD_Pad2.0mm
- renumbered R45 to R42, R46 to R43, R47 to R44, R50 to R45, R51 to R46, R52 to R47, U10 to U5, U12 to U6
Connections:
- net 3V3: now also R49.2, R52.2; no longer NT1.2, R45.2, U6.6 (VOUT)
- net 5V: now also R48.2, R51.2; no longer R42.2, U5.6 (VOUT)
- net GND: now also C38.2, C39.2, C40.2, R40.1, R41.1; no longer U5.2 (MODE), U6.2 (MODE)
- net VSYS: now also R39.2; no longer U5.1 (EN)
- net VSWREG_3V3_PG: now reaches U6.5 (PG)
- net VSWREG_3V3_PG: now also TP8.1
- net VSWREG_5V_PG: now reaches U5.5 (PG)
- net VSWREG_5V_PG: now also TP7.1
- net VCC renamed VPULLUP
- net VSWREG_FB renamed VSWREG_3V3_FB
- net VSWREG_3V3_FB: no longer R43.1, R44.2, U5.4 (FB)
- new net 3V3_PRE: C40.1, NT1.2, R45.2, R49.1, R53.2, U6.6 (VOUT)
- new net 5V_EN: R37.2
- new net 5V_PRE: C39.1, R42.2, R48.1, R50.2, U5.6 (VOUT)
- new net SNS_3V3_N: C42.1, R52.1, R56.1
- new net SNS_3V3_P: C42.2, R53.1, R57.1
- new net SNS_5V_N: C41.2, R51.1, R55.1
- new net SNS_5V_P: C41.1, R50.1, R54.1
- new net SWREG_MODE: R38.2, R40.2, U5.2 (MODE)
- new net VSWREG_3V3_MODE: R38.1, R41.2, U6.2 (MODE)
- new net VSWREG_5V_EN: C38.1, R37.1, R39.1, U5.1 (EN)
- new net VSWREG_5V_FB: R43.1, R44.2, U5.4 (FB)
- new net ~{SNS_EN}: R54.2, R55.2, R56.2, R57.2
- no-connect marks 2 -> 0
Other:
- note added: "* Select pull-up voltage in VCC_SEL."
- moved on the sheet: C36, C37, JP3, L2, L3, NT1, R42, R43, R44, R45, R46, R47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
