File: kicad/projects/mixpower-path-mini-bq25672-lv-board-r1/sheets/util-rgb.kicad_sch (KiCad schematic)
At the start: 7 parts, among them Q6 SI2101A, U7 SN74LV1T125DCK

Commit message: feat: small changes in schematics, some PCB routing
Parts:
- removed Q6: SI2101A, mixlib-generic-sot:SOT-323_SC-70, symbol mixlib-discrete-mosfet:SI2101A
- added Q5: PJE8405, mixlib-generic-sot:SOT-523, symbol mixlib-discrete-mosfet:PJE8405
Connections:
- net 5V: now also Q5.2 (S)
- net EN_G: now also Q5.1 (G)
- net VIN_RGB_LP: now also Q5.3 (D)
Changed lines of the file:
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@@
+	)
+	(symbol
+		(lib_id "mixlib-discrete-mosfet:PJE8405")
+		(at 91.44 72.39 270)
+		(mirror x)
+		(unit 1)
+		(exclude_from_sim no)
+		(in_bom yes)
+		(on_board yes)
+		(dnp no)
+		(property "Reference" "Q5"
+			(at 91.44 66.04 90)
+			(effects
+				(font
+					(size 1.27 1.27)
+				)
+			)
+		)
+		(property "Value" "PJE8405"
+			(at 91.44 68.58 90)
+			(effects
+				(font
+					(size 1.27 1.27)
+				)
+			)
+		)
+		(property "Footprint" "mixlib-generic-sot:SOT-523"
+			(at 86.106 71.12 0)
+			(effects
+				(font
+					(size 1.27 1.27)
+				)
+				(hide yes)
+			)
+		)
+		(property "Datasheet" "https://www.panjit.com.tw/upload/datasheet/PJE8405.pdf"
+			(at 86.868 72.39 0)
+			(effects
+				(font
+					(size 1.27 1.27)
+				)
+				(hide yes)
+			)
+		)
+		(property "Description" "30V 0.5A P-CHANNEL ENHANCEMENT MOSFET, SOT-523"
+			(at 85.344 71.882 0)
+			(effects
+				(font
+					(size 1.27 1.27)
+				)
+				(hide yes)
+			)
+		)
+		(pin "2"
+		)
+		(pin "3"
+		)
+		(pin "1"
+		)
+		(instances
+			(project "mixpower-path-mini-bq25672-lv-board-r1"
+				(path "/2e43857b-9bf9-460c-948c-ec2cf8a8d6b4/48666261-bb79-4da6-aeba-03c91aeede23"
+					(reference "Q5")
+					(unit 1)
+				)
+			)
+		)
 	)
 	(symbol
@@
 	)
 	(symbol
-		(lib_id "mixlib-discrete-mosfet:SI2101A")
-		(at 91.44 72.39 270)
-		(mirror x)
-		(unit 1)
-		(exclude_from_sim no)
-		(in_bom yes)
-		(on_board yes)
-		(dnp no)
-		(fields_autoplaced yes)
-		(property "Reference" "Q6"
-			(at 91.44 66.04 90)
-			(effects
-				(font
-					(size 1.27 1.27)
-				)
-			)
-		)
-		(property "Value" "SI2101A"
-			(at 91.44 68.58 90)
-			(effects
-				(font
-					(size 1.27 1.27)
-				)
-			)
-		)
-		(property "Footprint" "mixlib-generic-sot:SOT-323_SC-70"
-			(at 91.44 72.39 0)
-			(effects
-				(font
-					(size 1.27 1.27)
-				)
-				(hide yes)
-			)
-		)
-		(property "Datasheet" "https://www.mccsemi.com/pdf/products/SI2101A(SOT-323).pdf"
-			(at 91.44 72.39 0)
-			(effects
-				(font
-					(size 1.27 1.27)
-				)
-				(hide yes)
-			)
-		)
-		(property "Description" "20V 2A P-CHANNEL MOSFET, SOT-323 / SC-70"
-			(at 91.44 72.39 0)
-			(effects
-				(font
-					(size 1.27 1.27)
-				)
-				(hide yes)
-			)
-		)
-		(pin "1"
-		)
-		(pin "3"
-		)
-		(pin "2"
-		)
-		(instances
-			(project ""
-				(path "/2e43857b-9bf9-460c-948c-ec2cf8a8d6b4/48666261-bb79-4da6-aeba-03c91aeede23"
-					(reference "Q6")
-					(unit 1)
-				)
-			)
-		)
-	)
-	(symbol
 		(lib_id "power:GND")
 		(at 111.76 80.01 0)
@@
 		)
 		(instances
-			(project ""
+			(project "mixpower-path-mini-bq25672-lv-board-r1"
 				(path "/2e43857b-9bf9-460c-948c-ec2cf8a8d6b4/48666261-bb79-4da6-aeba-03c91aeede23"
 					(reference "U7")

Commit message: feat: failed PCB routing
Parts:
- removed C41: 100n, Capacitor_SMD:C_0402_1005Metric, symbol Device:C_Small
- removed Q5: PJE8405, mixlib-generic-sot:SOT-523, symbol mixlib-discrete-mosfet:PJE8405
- removed U7: SN74LV1T125DCK, Package_TO_SOT_SMD:SOT-353_SC-70-5, symbol Logic_LevelTranslator:SN74LV1T125DCK
- added Q8: DMG1029SVQ, mixlib-generic-sot:SOT-563, symbol mixlib-discrete-mosfet:DMG1029SVQ
- added R78: 4.7k, Resistor_SMD:R_0402_1005Metric, symbol Device:R_Small
- added R79: 1k, Resistor_SMD:R_0402_1005Metric, symbol Device:R_Small
- R76: renamed from R36; value 220 -> 1k
- renumbered C42 to C61, D7 to D8, R35 to R77
Connections:
- net 5V: now also Q8.4 (S2)
- net DI: now also Q8.1 (S1), R78.2
- net EN_G: now also Q8.5 (G2)
- net VIN_RGB_LP: now also Q8.3 (D2), R79.1
- net DI_TR: no longer names the net of D8.4 (DI)
- net DI_TR: now also Q8.6 (D1), R79.2
- new net 3V3_CS: Q8.2 (G1), R78.1
Other:
- moved on the sheet: C61, D8
