File: kicad/projects/mixpower-path-mini-bq25672-lv-board-r1/sheets/vpath-vdd1.kicad_sch (KiCad schematic)
At the start: 9 parts, among them U5 TPS22917DBV

Commit message: feat: failed PCB routing
Parts:
- removed C36, C38: 10u, Capacitor_SMD:C_0603_1608Metric, symbol Device:C_Small
- removed C37: 1u, Capacitor_SMD:C_0402_1005Metric, symbol Device:C_Small
- removed R31: 1M, Resistor_SMD:R_0402_1005Metric, symbol Device:R_Small
- added C58, C60: 10u, Capacitor_SMD:C_0402_1005Metric, symbol Device:C_Small
- R74: renamed from R33; value 1M -> 10M; now fitted
- renumbered C35 to C59, JP2 to JP5, R32 to R75, U5 to U10
Connections:
- net GND: now also C58.2, C60.2
- net VDD1_IN: now also C58.1
- net VOUT renamed VDD1
- net VDD1: now also C60.1
Other:
- moved on the sheet: C59, JP5
